Commit message: working grids\!

File: cvg_sim_gazebo/launch/grid.urdf (robot description, URDF)
Before this commit: robot grid, 1 links, 0 joints
Links:
- added link link1, mass 1.0; collision box size=1 1 0.1; visual box size=1 1 0.1
Joints:
- added joint base_to_link1: type fixed, parent base_link, child link1, origin xyz=0 0 0

Commit message: fixed grid color problem

File: cvg_sim_gazebo/launch/grid.urdf (robot description, URDF)
Before this commit: robot grid, 2 links, 1 joints
Links:
- added link link0, mass 1.0; collision box size=1 1 0.1; visual box size=1 1 0.1
- added link link2, mass 1.0; collision box size=1 1 0.1; visual box size=1 1 0.1
- added link link3, mass 1.0; collision box size=1 1 0.1; visual box size=1 1 0.1
- link base_link: mass 1.0 -> None; geometry 
Joints:
- added joint base_to_link0: type fixed, parent base_link, child link0, origin xyz=0 0 0
- added joint base_to_link2: type fixed, parent base_link, child link2, origin xyz=0 0 0
- added joint base_to_link3: type fixed, parent base_link, child link3, origin xyz=0 0 0
