Commit message: navigation changes

File: cvg_sim_gazebo/grid.urdf.xacro (robot description, xacro)
@@ -10,5 +10,5 @@
       <origin xyz="0 0 0"/>
       <geometry>
-        <box size="10 10 0.1" />
+        <box size="8 8 0.1" />
       </geometry>
     </visual>
@@ -16,5 +16,5 @@
       <origin xyz="0 0 0"/>
       <geometry>
-        <box size="10 10 0.1" />
+        <box size="8 8 0.1" />
       </geometry>
     </collision>
