Commit message: grid generation fix

File: cvg_sim_gazebo/urdf/grid.urdf.xacro (robot description, xacro)
@@ -10,5 +10,5 @@
       <origin xyz="0 0 0"/>
       <geometry>
-        <box size="8 8 0.1" />
+        <box size="6 6 0.1" />
       </geometry>
     </visual>
@@ -16,5 +16,5 @@
       <origin xyz="0 0 0"/>
       <geometry>
-        <box size="8 8 0.1" />
+        <box size="6 6 0.1" />
       </geometry>
     </collision>

Commit message: changed grid size and drone spawn location

File: cvg_sim_gazebo/urdf/grid.urdf.xacro (robot description, xacro)
@@ -10,5 +10,5 @@
       <origin xyz="0 0 0"/>
       <geometry>
-        <box size="6 6 0.1" />
+        <box size="10 10 0.1" />
       </geometry>
     </visual>
@@ -16,5 +16,5 @@
       <origin xyz="0 0 0"/>
       <geometry>
-        <box size="6 6 0.1" />
+        <box size="10 10 0.1" />
       </geometry>
     </collision>

Commit message: dynamic world generation

File: cvg_sim_gazebo/urdf/grid.urdf.xacro (robot description, xacro)
@@ -10,5 +10,5 @@
       <origin xyz="0 0 0"/>
       <geometry>
-        <box size="8 8 0.1" />
+        <box size="7 7 0.1" />
       </geometry>
     </visual>
@@ -16,5 +16,5 @@
       <origin xyz="0 0 0"/>
       <geometry>
-        <box size="8 8 0.1" />
+        <box size="7 7 0.1" />
       </geometry>
     </collision>

Commit message: kjfaskl

File: cvg_sim_gazebo/urdf/grid.urdf.xacro (robot description, xacro)
@@ -10,5 +10,5 @@
       <origin xyz="0 0 0"/>
       <geometry>
-        <box size="8 8 0.1" />
+        <box size="10 10 0.1" />
       </geometry>
     </visual>
@@ -16,5 +16,5 @@
       <origin xyz="0 0 0"/>
       <geometry>
-        <box size="8 8 0.1" />
+        <box size="10 10 0.1" />
       </geometry>
     </collision>
