Commit message: Undo my moron self

File: cvg_sim_gazebo/urdf/quadrotor.urdf.xacro (robot description, xacro)
@@ -6,5 +6,5 @@
     xmlns:xacro="http://playerstage.sourceforge.net/gazebo/xmlschema/#interface">
     <!-- Included URDF Files -->
-    <include filename="$(find tum_sim_gazebo)/urdf/quadrotor_base.urdf.xacro" />
+    <include filename="$(find cvg_sim_gazebo)/urdf/quadrotor_base.urdf.xacro" />
     <!-- Instantiate quadrotor_base_macro once (has no parameters atm) -->
     <quadrotor_base_macro />

File: cvg_sim_gazebo/urdf/quadrotor_base.urdf.xacro (robot description, xacro)
@@ -5,5 +5,5 @@
 xmlns:xacro="http://ros.org/wiki/xacro"
 >
-  <include filename="$(find tum_sim_gazebo_plugins)/urdf/quadrotor_plugins.urdf.xacro" />
+  <include filename="$(find cvg_sim_gazebo_plugins)/urdf/quadrotor_plugins.urdf.xacro" />
   <property name="pi" value="3.1415926535897931" />
   <!-- Main quadrotor link -->
@@ -18,5 +18,5 @@
         <origin xyz="0 0 0" rpy="0 0 0" />
         <geometry>
-          <mesh filename="package://tum_sim_gazebo/meshes/quadrotor/quadrotor_4.dae"/>
+          <mesh filename="package://cvg_sim_gazebo/meshes/quadrotor/quadrotor_4.dae"/>
         </geometry>
       </visual>
@@ -24,5 +24,5 @@
         <origin xyz="0 0 0" rpy="0 0 0" />
         <geometry>
-          <mesh filename="package://tum_sim_gazebo/meshes/quadrotor/quadrotor_4.stl"/>
+          <mesh filename="package://cvg_sim_gazebo/meshes/quadrotor/quadrotor_4.stl"/>
         </geometry>
       </collision>

File: cvg_sim_gazebo/urdf/quadrotor_sensors.urdf.xacro (robot description, xacro)
@@ -7,5 +7,5 @@
     <property name="M_PI" value="3.1415926535897931" />
     <!-- Included URDF Files -->
-    <include filename="$(find tum_sim_gazebo)/urdf/quadrotor_base.urdf.xacro" />
+    <include filename="$(find cvg_sim_gazebo)/urdf/quadrotor_base.urdf.xacro" />
     <!-- Instantiate quadrotor_base_macro once (has no parameters atm) -->
     <quadrotor_base_macro />
@@ -16,5 +16,5 @@
     </xacro:sonar_sensor>
     <!-- Hokuyo UTM-30LX mounted upside down below the quadrotor body
-    <include filename="$(find tum_sim_gazebo)/urdf/sensors/hokuyo_utm30lx.urdf.xacro" />
+    <include filename="$(find cvg_sim_gazebo)/urdf/sensors/hokuyo_utm30lx.urdf.xacro" />
     <xacro:hokuyo_utm30lx name="laser0" parent="base_link" ros_topic="scan" update_rate="40" ray_count="1081" min_angle="135" max_angle="-135">
       <origin xyz="0.0 0.0 0.08" rpy="${M_PI} 0 0"/>

File: cvg_sim_gazebo/urdf/quadrotor_sensors0.urdf (robot description, URDF)
Before this commit: robot quadrotor_hokuyo_utm30lx0, 6 links, 5 joints
Links:
- link base_link0: geometry collision mesh filename=package://cvg_sim_gazebo/meshes/quadrotor/quadrotor_4.stl; visual mesh filename=package://cvg_sim_gazebo/meshes/quadrotor/quadrotor_4.dae
- link sonar_link: geometry collision box size=0.01 0.01 0.01; visual mesh filename=package://cvg_sim_gazebo/meshes/sonar_sensor/max_sonar_ez4.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

File: cvg_sim_gazebo/urdf/quadrotor_sensors0.urdf.xacro (robot description, xacro)
@@ -7,14 +7,14 @@
     <property name="M_PI" value="3.1415926535897931" />
     <!-- Included URDF Files -->
-    <include filename="$(find tum_sim_gazebo)/urdf/quadrotor_base.urdf.xacro" />
+    <include filename="$(find cvg_sim_gazebo)/urdf/quadrotor_base.urdf.xacro" />
     <!-- Instantiate quadrotor_base_macro once (has no parameters atm) -->
     <quadrotor_base_macro />
     <!-- Sonar height sensor -->
-    <include filename="$(find tum_sim_gazebo)/urdf/sensors/sonar_sensor.urdf.xacro" />
+    <include filename="$(find cvg_sim_gazebo)/urdf/sensors/sonar_sensor.urdf.xacro" />
     <xacro:sonar_sensor name="sonar" parent="base_link" ros_topic="sonar_height" update_rate="10" min_range="0.01" max_range="3.0" field_of_view="40" ray_count="3">
       <origin xyz="-0.15 0.0 0.0" rpy="0 ${90*M_PI/180} 0"/>
     </xacro:sonar_sensor>
     <!-- Hokuyo UTM-30LX mounted upside down below the quadrotor body
-    <include filename="$(find tum_sim_gazebo)/urdf/sensors/hokuyo_utm30lx.urdf.xacro" />
+    <include filename="$(find cvg_sim_gazebo)/urdf/sensors/hokuyo_utm30lx.urdf.xacro" />
     <xacro:hokuyo_utm30lx name="laser0" parent="base_link" ros_topic="scan" update_rate="40" ray_count="1081" min_angle="135" max_angle="-135">
       <origin xyz="0.0 0.0 0.08" rpy="${M_PI} 0 0"/>
@@ -22,10 +22,10 @@
     <!-- The following two cameras should be united to one! -->
     <!-- Forward facing camera -->
-    <include filename="$(find tum_sim_gazebo)/urdf/sensors/generic_camera.urdf.xacro" />
+    <include filename="$(find cvg_sim_gazebo)/urdf/sensors/generic_camera.urdf.xacro" />
     <xacro:generic_camera name="front" sim_name="ardrone" parent="base_link" update_rate="60" res_x="640" res_y="360" image_format="R8G8B8" hfov="81">
       <origin xyz="0.21 0.0 0.01" rpy="0 0 0"/>
     </xacro:generic_camera>
     <!-- Downward facing camera -->
-    <include filename="$(find tum_sim_gazebo)/urdf/sensors/generic_camera.urdf.xacro" />
+    <include filename="$(find cvg_sim_gazebo)/urdf/sensors/generic_camera.urdf.xacro" />
     <xacro:generic_camera name="bottom" sim_name="ardrone" parent="base_link" update_rate="60" res_x="640" res_y="360" image_format="R8G8B8" hfov="81">
       <origin xyz="0.15 0.0 0.0" rpy="0 -${M_PI/2} 0"/>

File: cvg_sim_gazebo/urdf/quadrotor_sensors1.urdf (robot description, URDF)
Before this commit: robot quadrotor_hokuyo_utm30lx1, 6 links, 5 joints
Links:
- link base_link1: geometry collision mesh filename=package://cvg_sim_gazebo/meshes/quadrotor/quadrotor_4.stl; visual mesh filename=package://cvg_sim_gazebo/meshes/quadrotor/quadrotor_4.dae
- link sonar_link: geometry collision box size=0.01 0.01 0.01; visual mesh filename=package://cvg_sim_gazebo/meshes/sonar_sensor/max_sonar_ez4.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

File: cvg_sim_gazebo/urdf/quadrotor_sensors1.urdf.xacro (robot description, xacro)
@@ -7,14 +7,14 @@
     <property name="M_PI" value="3.1415926535897931" />
     <!-- Included URDF Files -->
-    <include filename="$(find tum_sim_gazebo)/urdf/quadrotor_base.urdf.xacro" />
+    <include filename="$(find cvg_sim_gazebo)/urdf/quadrotor_base.urdf.xacro" />
     <!-- Instantiate quadrotor_base_macro once (has no parameters atm) -->
     <quadrotor_base_macro />
     <!-- Sonar height sensor -->
-    <include filename="$(find tum_sim_gazebo)/urdf/sensors/sonar_sensor.urdf.xacro" />
+    <include filename="$(find cvg_sim_gazebo)/urdf/sensors/sonar_sensor.urdf.xacro" />
     <xacro:sonar_sensor name="sonar" parent="base_link" ros_topic="sonar_height" update_rate="10" min_range="0.01" max_range="3.0" field_of_view="40" ray_count="3">
       <origin xyz="-0.15 0.0 0.0" rpy="0 ${90*M_PI/180} 0"/>
     </xacro:sonar_sensor>
     <!-- Hokuyo UTM-30LX mounted upside down below the quadrotor body
-    <include filename="$(find tum_sim_gazebo)/urdf/sensors/hokuyo_utm30lx.urdf.xacro" />
+    <include filename="$(find cvg_sim_gazebo)/urdf/sensors/hokuyo_utm30lx.urdf.xacro" />
     <xacro:hokuyo_utm30lx name="laser0" parent="base_link" ros_topic="scan" update_rate="40" ray_count="1081" min_angle="135" max_angle="-135">
       <origin xyz="0.0 0.0 0.08" rpy="${M_PI} 0 0"/>
@@ -22,10 +22,10 @@
     <!-- The following two cameras should be united to one! -->
     <!-- Forward facing camera -->
-    <include filename="$(find tum_sim_gazebo)/urdf/sensors/generic_camera.urdf.xacro" />
+    <include filename="$(find cvg_sim_gazebo)/urdf/sensors/generic_camera.urdf.xacro" />
     <xacro:generic_camera name="front" sim_name="ardrone" parent="base_link" update_rate="60" res_x="640" res_y="360" image_format="R8G8B8" hfov="81">
       <origin xyz="0.21 0.0 0.01" rpy="0 0 0"/>
     </xacro:generic_camera>
     <!-- Downward facing camera -->
-    <include filename="$(find tum_sim_gazebo)/urdf/sensors/generic_camera.urdf.xacro" />
+    <include filename="$(find cvg_sim_gazebo)/urdf/sensors/generic_camera.urdf.xacro" />
     <xacro:generic_camera name="bottom" sim_name="ardrone" parent="base_link" update_rate="60" res_x="640" res_y="360" image_format="R8G8B8" hfov="81">
       <origin xyz="0.15 0.0 0.0" rpy="0 -${M_PI/2} 0"/>

File: cvg_sim_gazebo/urdf/quadrotor_sensors2.urdf (robot description, URDF)
Before this commit: robot quadrotor_hokuyo_utm30lx2, 6 links, 5 joints
Links:
- link base_link2: geometry collision mesh filename=package://cvg_sim_gazebo/meshes/quadrotor/quadrotor_4.stl; visual mesh filename=package://cvg_sim_gazebo/meshes/quadrotor/quadrotor_4.dae
- link sonar_link: geometry collision box size=0.01 0.01 0.01; visual mesh filename=package://cvg_sim_gazebo/meshes/sonar_sensor/max_sonar_ez4.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

File: cvg_sim_gazebo/urdf/quadrotor_sensors2.urdf.xacro (robot description, xacro)
@@ -7,14 +7,14 @@
     <property name="M_PI" value="3.1415926535897931" />
     <!-- Included URDF Files -->
-    <include filename="$(find tum_sim_gazebo)/urdf/quadrotor_base.urdf.xacro" />
+    <include filename="$(find cvg_sim_gazebo)/urdf/quadrotor_base.urdf.xacro" />
     <!-- Instantiate quadrotor_base_macro once (has no parameters atm) -->
     <quadrotor_base_macro />
     <!-- Sonar height sensor -->
-    <include filename="$(find tum_sim_gazebo)/urdf/sensors/sonar_sensor.urdf.xacro" />
+    <include filename="$(find cvg_sim_gazebo)/urdf/sensors/sonar_sensor.urdf.xacro" />
     <xacro:sonar_sensor name="sonar" parent="base_link" ros_topic="sonar_height" update_rate="10" min_range="0.01" max_range="3.0" field_of_view="40" ray_count="3">
       <origin xyz="-0.15 0.0 0.0" rpy="0 ${90*M_PI/180} 0"/>
     </xacro:sonar_sensor>
     <!-- Hokuyo UTM-30LX mounted upside down below the quadrotor body
-    <include filename="$(find tum_sim_gazebo)/urdf/sensors/hokuyo_utm30lx.urdf.xacro" />
+    <include filename="$(find cvg_sim_gazebo)/urdf/sensors/hokuyo_utm30lx.urdf.xacro" />
     <xacro:hokuyo_utm30lx name="laser0" parent="base_link" ros_topic="scan" update_rate="40" ray_count="1081" min_angle="135" max_angle="-135">
       <origin xyz="0.0 0.0 0.08" rpy="${M_PI} 0 0"/>
@@ -22,10 +22,10 @@
     <!-- The following two cameras should be united to one! -->
     <!-- Forward facing camera -->
-    <include filename="$(find tum_sim_gazebo)/urdf/sensors/generic_camera.urdf.xacro" />
+    <include filename="$(find cvg_sim_gazebo)/urdf/sensors/generic_camera.urdf.xacro" />
     <xacro:generic_camera name="front" sim_name="ardrone" parent="base_link" update_rate="60" res_x="640" res_y="360" image_format="R8G8B8" hfov="81">
       <origin xyz="0.21 0.0 0.01" rpy="0 0 0"/>
     </xacro:generic_camera>
     <!-- Downward facing camera -->
-    <include filename="$(find tum_sim_gazebo)/urdf/sensors/generic_camera.urdf.xacro" />
+    <include filename="$(find cvg_sim_gazebo)/urdf/sensors/generic_camera.urdf.xacro" />
     <xacro:generic_camera name="bottom" sim_name="ardrone" parent="base_link" update_rate="60" res_x="640" res_y="360" image_format="R8G8B8" hfov="81">
       <origin xyz="0.15 0.0 0.0" rpy="0 -${M_PI/2} 0"/>

File: cvg_sim_gazebo/urdf/sensors/hokuyo_utm30lx.urdf.xacro (robot description, xacro)
@@ -20,5 +20,5 @@
 	  <origin xyz="0 0 0" rpy="0 0 0" />
           <geometry>
-          <mesh filename="package://tum_sim_gazebo/meshes/hokuyo_utm30lx/hokuyo_utm_30lx$(optenv TEST_SELF_FILTER).dae"/>
+          <mesh filename="package://cvg_sim_gazebo/meshes/hokuyo_utm30lx/hokuyo_utm_30lx$(optenv TEST_SELF_FILTER).dae"/>
         </geometry>
 	</visual>

File: cvg_sim_gazebo/urdf/sensors/sonar_sensor.urdf.xacro (robot description, xacro)
@@ -21,5 +21,5 @@
         <geometry>
           <!--<box size="0.01 0.01 0.01" /> -->
-          <mesh filename="package://tum_sim_gazebo/meshes/sonar_sensor/max_sonar_ez4.dae"/>
+          <mesh filename="package://cvg_sim_gazebo/meshes/sonar_sensor/max_sonar_ez4.dae"/>
         </geometry>
       </visual>

File: cvg_sim_gazebo_plugins/urdf/quadrotor_plugins.urdf.xacro (robot description, xacro)
@@ -1,6 +1,6 @@
 <?xml version="1.0"?>
 <robot xmlns:xacro="http://ros.org/wiki/xacro">
-  <xacro:include filename="$(find tum_sim_gazebo_plugins)/urdf/quadrotor_sensors.urdf.xacro" />
-  <xacro:include filename="$(find tum_sim_gazebo_plugins)/urdf/quadrotor_simple_controller.urdf.xacro" />
+  <xacro:include filename="$(find cvg_sim_gazebo_plugins)/urdf/quadrotor_sensors.urdf.xacro" />
+  <xacro:include filename="$(find cvg_sim_gazebo_plugins)/urdf/quadrotor_simple_controller.urdf.xacro" />
   <!-- Quadrotor Gazebo Plugins -->
   <xacro:macro name="quadrotor_plugins">

Commit message: Got cameras working, still can't cantrol drones though
it seems the plugins are interfering with each other

File: cvg_sim_gazebo/urdf/quadrotor.urdf.xacro (robot description, xacro)
@@ -9,3 +9,24 @@
     <!-- Instantiate quadrotor_base_macro once (has no parameters atm) -->
     <quadrotor_base_macro />
+    <!-- Sonar height sensor -->
+    <include filename="$(find cvg_sim_gazebo)/urdf/sensors/sonar_sensor.urdf.xacro" />
+    <xacro:sonar_sensor name="sonar" parent="base_link" ros_topic="sonar_height" update_rate="10" min_range="0.01" max_range="3.0" field_of_view="${40*M_PI/180}" ray_count="3">
+      <origin xyz="-0.15 0.0 0.0" rpy="0 ${90*M_PI/180} 0"/>
+    </xacro:sonar_sensor>
+    <!-- Hokuyo UTM-30LX mounted upside down below the quadrotor body
+    <include filename="$(find cvg_sim_gazebo)/urdf/sensors/hokuyo_utm30lx.urdf.xacro" />
+    <xacro:hokuyo_utm30lx name="laser0" parent="base_link" ros_topic="scan" update_rate="40" ray_count="1081" min_angle="135" max_angle="-135">
+      <origin xyz="0.0 0.0 0.08" rpy="${M_PI} 0 0"/>
+    </xacro:hokuyo_utm30lx>-->
+    <!-- The following two cameras should be united to one! -->
+    <!-- Forward facing camera -->
+    <include filename="$(find cvg_sim_gazebo)/urdf/sensors/generic_camera.urdf.xacro" />
+    <xacro:generic_camera name="front" parent="base_link" update_rate="60" res_x="640" res_y="360" image_format="R8G8B8" hfov="${81*M_PI/180}">
+      <origin xyz="0.21 0.0 0.01" rpy="0 0 0"/>
+    </xacro:generic_camera>
+    <!-- Downward facing camera -->
+    <include filename="$(find cvg_sim_gazebo)/urdf/sensors/generic_camera.urdf.xacro" />
+    <xacro:generic_camera name="bottom" parent="base_link" update_rate="60" res_x="640" res_y="360" image_format="R8G8B8" hfov="${81*M_PI/180}">
+      <origin xyz="0.15 0.0 0.0" rpy="0 -${M_PI/2} 0"/>
+    </xacro:generic_camera>
 </robot>

File: cvg_sim_gazebo/urdf/sensors/generic_camera.urdf.xacro (robot description, xacro)
@@ -6,5 +6,5 @@
   >
     <property name="M_PI" value="3.1415926535897931" />
-    <xacro:macro name="generic_camera" params="name sim_name parent *origin update_rate res_x res_y image_format hfov">
+    <xacro:macro name="generic_camera" params="name parent *origin update_rate res_x res_y image_format hfov">
       <joint name="${name}_joint" type="fixed">
         <insert_block name="origin" />
@@ -13,9 +13,4 @@
       </joint>
       <link name="${name}_link">
-        <inertial>
-          <mass value="0.001" />
-          <origin xyz="0 0 0" rpy="0 0 0" />
-          <inertia ixx="0.0001" ixy="0" ixz="0" iyy="0.0001" iyz="0" izz="0.0001" />
-        </inertial>
         <visual>
           <origin xyz="0 0 0" rpy="0 0 0" />
@@ -27,37 +22,11 @@
     </material>
         </visual>
-        <collision>
+        <!--<collision>
           <origin xyz="0 0 0" rpy="0 0 0" />
           <geometry>
             <box size="0.01 0.01 0.01" />
           </geometry>
-        </collision>
+        </collision>-->
       </link>
-    <joint name="${name}_optical_joint" type="fixed">
-      <origin xyz="0 0 0" rpy="${-M_PI/2} 0.0 ${-M_PI/2}" />
-      <parent link="${name}_link" />
-      <child link="ardrone_base_${name}cam"/>
-    </joint>
-    <link name="ardrone_base_${name}cam">
-      <inertial>
-        <mass value="0.01" />
-        <origin xyz="0 0 0" />
-        <inertia ixx="0.001"  ixy="0.0"  ixz="0.0"
-                 iyy="0.001"  iyz="0.0"
-                 izz="0.001" />
-      </inertial>
-      <visual>
-        <origin xyz="0 0 0" rpy="0 0 0"/>
-        <geometry>
-          <box size="0.001 0.001 0.001" />
-        </geometry>
-      </visual>
-      <collision>
-        <origin xyz="0 0 0" rpy="0 0 0"/>
-        <geometry>
-          <box size="0.001 0.001 0.001" />
-        </geometry>
-      </collision>
-    </link>
     <gazebo reference="${name}_link">
       <sensor type="camera" name="${name}_camera_sensor">
@@ -70,5 +39,5 @@
             <format>${image_format}</format>
           </image>
-          <clip>0.01
+          <clip>
 	    <near>0.01</near>
             <far>100</far>
@@ -76,14 +45,12 @@
         </camera>
         <plugin name="${name}_camera_controller" filename="libgazebo_ros_camera.so">
-	  <cameraName>${name}</cameraName>
+	  <cameraName>ardrone/${name}</cameraName>
           <alwaysOn>true</alwaysOn>
           <updateRate>${update_rate}</updateRate>
-          <imageTopicName>${name}/image_raw</imageTopicName>
-          <cameraInfoTopicName>${name}/camera_info</cameraInfoTopicName>
+          <imageTopicName>image_raw</imageTopicName>
+          <cameraInfoTopicName>camera_info</cameraInfoTopicName>
           <frameName>ardrone_base_${name}cam</frameName>
         </plugin>
       </sensor>
-      <turnGravityOff>true</turnGravityOff>
-      <material>PR2/Blue</material>
     </gazebo>
     </xacro:macro>

File: cvg_sim_gazebo/urdf/sensors/sonar_sensor.urdf.xacro (robot description, xacro)
@@ -12,9 +12,4 @@
     </joint>
     <link name="${name}_link">
-      <inertial>
-        <mass value="0.001" />
-        <origin xyz="0 0 0" rpy="0 0 0" />
-        <inertia ixx="0.000000017" ixy="0" ixz="0" iyy="0.000000017" iyz="0" izz="0.000000017" />
-      </inertial>
       <visual>
         <origin xyz="0 0 0" rpy="0 0 0" />
@@ -24,10 +19,4 @@
         </geometry>
       </visual>
-      <collision>
-        <origin xyz="0 0 0" rpy="0 0 0" />
-        <geometry>
-          <box size="0.01 0.01 0.01" />
-        </geometry>
-      </collision>
     </link>
     <gazebo reference="${name}_link">
@@ -57,4 +46,7 @@
           <topicName>${ros_topic}</topicName>
           <frameId>${name}_link</frameId>
+	<offset>0.0</offset>
+	<drift>0.0</drift>
+	<driftFrequency>0.0</driftFrequency>
         </plugin>
       </sensor>
