Commit message: Change weight of drone to match reality

File: thinc_sim_gazebo/urdf/quadrotor_base.urdf.xacro (robot description, xacro)
@@ -11,5 +11,5 @@
     <link name="base_link">
       <inertial>
-        <mass value="1.477" />
+        <mass value="0.437" />
         <origin xyz="0 0 0" />
         <inertia ixx="0.01152" ixy="0.0" ixz="0.0" iyy="0.01152" iyz="0.0" izz="0.0218" />
