Commit message: Continue rebranding

File: thinc_sim_gazebo/urdf/sensors/hokuyo_utm30lx.urdf.xacro (robot description, xacro)
@@ -27,5 +27,5 @@
           <geometry>
           <box size="0.058 0.058 0.087" />
-          <!--<mesh filename="package://hector_sensors_description/meshes/hokuyo_utm30lx/hokuyo_utm_30lx.stl"/>-->
+          <!--<mesh filename="package://thinc_sensors_description/meshes/hokuyo_utm30lx/hokuyo_utm_30lx.stl"/>-->
         </geometry>
 	</collision>

File: thinc_sim_gazebo/urdf/sensors/sonar_sensor.urdf.xacro (robot description, xacro)
@@ -42,5 +42,5 @@
           </scan>
         </ray>
-        <plugin name="gazebo_ros_${name}_controller" filename="libhector_gazebo_ros_sonar.so">
+        <plugin name="gazebo_ros_${name}_controller" filename="libthinc_gazebo_ros_sonar.so">
           <gaussianNoise>0.000</gaussianNoise>
           <topicName>${ros_topic}</topicName>

File: thinc_sim_gazebo_plugins/urdf/quadrotor_sensors.urdf.xacro (robot description, xacro)
@@ -10,5 +10,5 @@
   <xacro:macro name="quadrotor_sensors">
     <gazebo>
-      <plugin name="quadrotor_imu_sim" filename="libhector_gazebo_ros_imu.so">
+      <plugin name="quadrotor_imu_sim" filename="libthinc_gazebo_ros_imu.so">
         <alwaysOn>true</alwaysOn>
         <updateRate>100.0</updateRate>
@@ -26,5 +26,5 @@
         <headingGaussianNoise>0.00</headingGaussianNoise>
       </plugin>
-      <plugin name="quadrotor_baro_sim" filename="libhector_gazebo_ros_baro.so">
+      <plugin name="quadrotor_baro_sim" filename="libthinc_gazebo_ros_baro.so">
         <alwaysOn>true</alwaysOn>
         <updateRate>10.0</updateRate>
@@ -37,5 +37,5 @@
         <gaussianNoise>0.5</gaussianNoise>
       </plugin>
-      <plugin name="quadrotor_magnetic_sim" filename="libhector_gazebo_ros_magnetic.so">
+      <plugin name="quadrotor_magnetic_sim" filename="libthinc_gazebo_ros_magnetic.so">
         <alwaysOn>true</alwaysOn>
         <updateRate>10.0</updateRate>
@@ -47,5 +47,5 @@
         <gaussianNoise>1.3e-2 1.3e-2 1.3e-2</gaussianNoise>
       </plugin>
-      <plugin name="quadrotor_gps_sim" filename="libhector_gazebo_ros_gps.so">
+      <plugin name="quadrotor_gps_sim" filename="libthinc_gazebo_ros_gps.so">
         <alwaysOn>true</alwaysOn>
         <updateRate>4.0</updateRate>

File: thinc_sim_gazebo_plugins/urdf/quadrotor_simple_controller.urdf.xacro (robot description, xacro)
@@ -7,5 +7,5 @@
   <xacro:macro name="quadrotor_controller">
     <gazebo>
-      <plugin name="quadrotor_simple_controller" filename="libhector_gazebo_quadrotor_simple_controller.so">
+      <plugin name="quadrotor_simple_controller" filename="libthinc_gazebo_quadrotor_simple_controller.so">
         <robotNamespace>$(arg namespace)</robotNamespace>
         <alwaysOn>true</alwaysOn>
@@ -32,5 +32,5 @@
         <motionDriftNoiseTime>5.0</motionDriftNoiseTime>
       </plugin>
-      <plugin name="quadrotor_state_controller" filename="libhector_gazebo_quadrotor_state_controller.so">
+      <plugin name="quadrotor_state_controller" filename="libthinc_gazebo_quadrotor_state_controller.so">
         <robotNamespace>$(arg namespace)</robotNamespace>
         <alwaysOn>true</alwaysOn>
